Commit message: Added the arms base and modified the initial pose of the arms

File: pybullet_controller/URDFs/arms_base/arms_base.urdf (robot description, URDF)
Before this commit: robot arms_base, 1 links, 0 joints
Links:
- link baseLink: geometry collision box size=0.08 0.02 1.5; collision box size=0.365 0.455 0.05
