Commit message: Stable demo mode

File: pybullet_controller/URDFs/cube_and_square/cube_box_2.urdf (robot description, URDF)
Before this commit: robot cube.urdf, 1 links, 0 joints
Links:
- link baseLink: mass .50 -> 50; geometry collision box size=.74 1.8 .73; visual mesh filename=cube.obj scale=.74 1.8 .73

File: pybullet_controller/URDFs/cylinder/cylinder.urdf (robot description, URDF)
Before this commit: robot cylinder, 1 links, 0 joints
Links:
- link baseLink: mass 1.0 -> 0.380; geometry collision mesh filename=cylinder.obj scale=1.0 1.0 1.0; visual mesh filename=cylinder.obj scale=1.0 1.0 1.0
